File: schematics/nerf-light.kicad_sch (KiCad schematic)
At the start: 3 parts, among them M1 Motor_Servo, U1 SC0194_9_

Commit message: docs: Add wiring diagram
Parts:
- removed A1: Pololu_Breakout_A4988, Module:Pololu_Breakout-16_15.2x20.3mm, symbol Driver_Motor:Pololu_Breakout_A4988
- added D1, D2: LED, symbol Device:LED
- added R1, R2: 400, symbol Device:R
- added SW1: SW_Push, symbol Switch:SW_Push
Connections:
- net GND: now also D1.1 (K), D2.1 (K), SW1.1
- net at U1.16 (GPIO23/GPIO_GEN4): now also R1.2
- net at U1.18 (GPIO24/GPIO_GEN5): now also R2.2
- net at U1.22 (GPIO25/GPIO_GEN6): now also SW1.2
- new net: D1.2 (A), R1.1
- new net: D2.2 (A), R2.1
